File: hardware/FailDeadly/FailDeadly.kicad_pcb (KiCad board)
At the start: 4 copper layers, 70 x 25 mm, 101 parts, among them IC1 MT9700, IC2 SN74LVC2G02DCUR, J1 KLS1-180B-W, J2 ionister_conn, J3 EXTERNAL_RESET, J4 Conn_02x04_Odd_Even, Q4 IRLML6401, Q5 IRLML6401, Q6 IRLML6401, U1 USBLC6-2P6, U2 AP2112K-3.3, U3 LTV-817S, U4 STM32F401CCUx, U5 SN74LVC1G14DBV, U6 MCP121T-270E_TT, U7 SN74LVC1G14DBV, U8 SN74LVC1G17DBVRE4, Y1 KX-9A 24Mhz

Commit message: Small changes in schematic
The crystal oscillator was changed from 24 MHz to 25 MHz so that the original board and the STM32 Green Pill (test board) were compatible in the oscillator configuration in the firmware.
Parts:
- Y1: value KX-9A 24Mhz -> KX-9A 25Mhz
Changed lines of the file:
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@@
 			)
 		)
-		(property "Value" "KX-9A 24Mhz"
+		(property "Value" "KX-9A 25Mhz"
 			(at 0 0 90)
 			(layer "F.SilkS")
@@
 	)
 	(segment
+		(start 110.31 120.5)
+		(end 112.19 120.5)
+		(width 0.25)
+		(layer "F.Cu")
+		(net "Net-(U2-EN)")
+	)
+	(segment
+		(start 114 119.8)
+		(end 112.91 119.8)
+		(width 0.25)
+		(layer "F.Cu")
+		(net "Net-(U2-EN)")
+	)
+	(segment
+		(start 112.91 119.8)
+		(end 112.2 120.51)
+		(width 0.25)
+		(layer "F.Cu")
+		(net "Net-(U2-EN)")
+	)
+	(segment
+		(start 112.19 120.5)
+		(end 112.2 120.51)
+		(width 0.25)
+		(layer "F.Cu")
+		(net "Net-(U2-EN)")
+	)
+	(segment
+		(start 110.21 120.4)
+		(end 110.31 120.5)
+		(width 0.25)
+		(layer "F.Cu")
+		(net "Net-(U2-EN)")
+	)
+	(segment
 		(start 121.55 117.5)
 		(end 121.55 117.875)
@@
 		(net "Net-(S1-OUTPUT)")
 	)
-	(segment
-		(start 110.31 120.5)
-		(end 112.19 120.5)
-		(width 0.25)
-		(layer "F.Cu")
-		(net "Net-(U2-EN)")
-	)
-	(segment
-		(start 114 119.8)
-		(end 112.91 119.8)
-		(width 0.25)
-		(layer "F.Cu")
-		(net "Net-(U2-EN)")
-	)
-	(segment
-		(start 112.91 119.8)
-		(end 112.2 120.51)
-		(width 0.25)
-		(layer "F.Cu")
-		(net "Net-(U2-EN)")
-	)
-	(segment
-		(start 112.19 120.5)
-		(end 112.2 120.51)
-		(width 0.25)
-		(layer "F.Cu")
-		(net "Net-(U2-EN)")
-	)
-	(segment
-		(start 110.21 120.4)
-		(end 110.31 120.5)
-		(width 0.25)
-		(layer "F.Cu")
-		(net "Net-(U2-EN)")
-	)
 	(zone
