File: hardware/FailDeadly/MCU.kicad_sch (KiCad schematic)
At the start: 32 parts, among them J4 Conn_02x04_Odd_Even, Q4 IRLML6401, U4 STM32F401CCUx, U6 MCP121T-270E_TT, U7 SN74LVC1G14DBV, Y1 KX-9A 24Mhz

Commit message: Small changes in schematic
The crystal oscillator was changed from 24 MHz to 25 MHz so that the original board and the STM32 Green Pill (test board) were compatible in the oscillator configuration in the firmware.
Parts:
- Y1: value KX-9A 24Mhz -> KX-9A 25Mhz
Changed lines of the file:
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@@
 		(title "MCU")
 		(date "2026-07-20")
-		(rev "001")
+		(rev "002")
 	)
 	(rectangle
@@
 			)
 		)
-		(property "Value" "KX-9A 24Mhz"
+		(property "Value" "KX-9A 25Mhz"
 			(at 181.61 85.09 0)
 			(show_name no)
